Commit message: 36

File: install/mazebot/share/mazebot/urdf/mazebot.urdf (robot description, URDF)
Before this commit: robot mazebot, 5 links, 4 joints
Links:
- added link camera_link; visual box size=0.05 0.04 0.05
Joints:
- added joint camera_joint: type fixed, parent base_footprint, child camera_link, origin xyz=-0.32 0.0 0.14 rpy=0.0 0.0 0.0, axis 0 0 1
- joint laser_joint: origin xyz=-0.32 0.0 0.08 rpy=0.0 0.0 3.14 -> xyz=-0.32 0.0 0.08 rpy=0.0 0.0 0.0

Commit message: maze world import

File: install/mazebot/share/mazebot/urdf/mazebot.urdf (robot description, URDF)
Before this commit: robot mazebot, 6 links, 5 joints
Joints:
- joint laser_joint: origin xyz=-0.32 0.0 0.08 rpy=0.0 0.0 0.0 -> xyz=-0.32 0.0 0.08 rpy=0.0 0.0 3.14
